Commit message: wheels added

File: mino_description/urdf/include/common_macros.urdf.xacro (robot description, xacro)
@@ -1,13 +1,10 @@
 <?xml version="1.0"?>
 <robot xmlns:xacro="http://www.ros.org/wiki/xacro">
+<!--           Include materials            -->
+<xacro:include filename="./materials.urdf.xacro"/>
+<!--########################################-->
 <!--               Base xacro               -->
 <xacro:macro name="base"
     params="link_name:='base_link' base_prop mesh:='' scale:=''">
-    <link name="footprint"/>
-    <joint name="footprint_to_base" type="fixed">
-        <parent link="footprint"/>
-        <child link="base_link"/>
-        <origin xyz="-0.1 0 0"/>
-    </joint>
     <link name="${link_name}">
     <!-- if no 3d model -->
@@ -18,4 +15,5 @@
                 <box size="${base_prop['x_size']} ${base_prop['y_size']} ${base_prop['z_size']}"/>
             </geometry>
+            <material name="blue"/>
         </visual>
     </xacro:if>
@@ -29,3 +27,76 @@
 </xacro:macro>
 <!--########################################-->
+<!--            Footprint xacro              -->
+<xacro:macro name="footprint"
+    params="wheel_props">
+    <link name="base_footprint"/>
+    <joint name="base_to_footprint_joint" type="fixed">
+        <parent link="base_link"/>
+        <child link="base_footprint"/>
+        <origin xyz="0.0 0.0 ${-(wheel_props['radius']) + wheel_props['z_offset']}" rpy="0.0 0.0 0.0"/>
+    </joint>
+</xacro:macro>
+<!--######################################## -->
+<!--               Wheel xacro               -->
+<xacro:macro name="wheel"
+    params="prefix reflect wheel_props base_props">
+<xacro:property name="pos_x_joint"
+    value="${(base_props['x_size']/2) - wheel_props['x_offset']}"/>
+<xacro:property name="pos_y_joint"
+    value="${(base_props['y_size']/2) + wheel_props['y_offset'] + (wheel_props['length']/2)}"/>
+<xacro:property name="pos_z_joint" value="${wheel_props['z_offset']}"/>
+    <link name="${prefix}_wheel">
+    <!-- if no 3d model -->
+    <xacro:if value="${wheel_props['mesh'] == ''}">
+        <visual>
+            <origin xyz="0.0 0.0 0.0" rpy="${pi/2} 0.0 0.0"/>
+            <geometry>
+                <cylinder radius="${wheel_props['radius']}" length="${wheel_props['length']}"/>
+            </geometry>
+            <material name="black"/>
+        </visual>
+    </xacro:if>
+        <collision>
+            <origin xyz="0.0 0.0 0.0" rpy="${pi/2} 0.0 0.0"/>
+            <geometry>
+                <cylinder radius="${wheel_props['radius']}" length="${wheel_props['length']}"/>
+            </geometry>
+        </collision>
+    </link>
+    <joint name="${prefix}_wheel_joint" type="continuous">
+        <axis xyz="0.0 1.0 0.0" rpy="0.0 0.0 0.0"/>
+        <parent link="base_link"/>
+        <child link="${prefix}_wheel"/>
+        <origin xyz="${pos_x_joint} ${reflect * pos_y_joint} ${pos_z_joint}" rpy="0.0 0.0 0.0"/>
+    </joint>
+</xacro:macro>
+<!--########################################-->
+<!--               Caster xacro               -->
+<xacro:macro name="caster"
+    params="link_name:='caster_link' caster_props">
+    <link name="${link_name}">
+    <xacro:if value="${caster_props['mesh'] == ''}">
+        <visual>
+            <origin xyz="0.0 0.0 0.0" rpy="0.0 0.0 0.0"/>
+            <geometry>
+                <sphere radius="${caster_props['radius']}"/>
+            </geometry>
+            <material name="green"/>
+        </visual>
+        <collision>
+            <origin xyz="0.0 0.0 0.0" rpy="0.0 0.0 0.0"/>
+            <geometry>
+                <sphere radius="${caster_props['radius']}"/>
+            </geometry>
+        </collision>
+    </xacro:if>
+    </link>
+    <joint name="$caster_joint" type="fixed">
+        <parent link="base_link"/>
+        <child link="${link_name}"/>
+        <origin xyz="${caster_props['x_offset']} ${caster_props['y_offset']} ${caster_props['z_offset']}"
+                rpy="0.0 0.0 0.0"/>
+    </joint>
+</xacro:macro>
+<!--##########################################-->
 </robot>

File: mino_description/urdf/mino.urdf.xacro (robot description, xacro)
@@ -12,6 +12,19 @@
     <xacro:property name="base_yaml" value="$(arg config_dir)/base.yaml"/>
     <xacro:property name="base_props" value="${xacro.load_yaml(base_yaml)}"/>
+    <xacro:property name="wheel_yaml" value="$(arg config_dir)/wheels.yaml"/>
+    <xacro:property name="wheel_props" value="${xacro.load_yaml(wheel_yaml)}"/>
+    <xacro:property name="caster_yaml" value="$(arg config_dir)/caster.yaml"/>
+    <xacro:property name="caster_props" value="${xacro.load_yaml(caster_yaml)}"/>
     <!-- ########################################## -->
+    <!-- Footprint link-->
+    <xacro:footprint wheel_props="${wheel_props}"/>
     <!-- Base link -->
     <xacro:base link_name="base_link" base_prop="${base_props}" mesh="${base_props['mesh']}"/>
+    <!-- Wheels links -->
+    <xacro:wheel prefix="right" reflect="-1" wheel_props="${wheel_props}" base_props="${base_props}"/>
+    <xacro:wheel prefix="left" reflect="1" wheel_props="${wheel_props}" base_props="${base_props}"/>
+    <!-- Caster wheel link -->
+    <xacro:caster link_name="caster_link" caster_props="${caster_props}"/>
+    <!-- Sensor link -->
+    <!-- ros2_control -->
 </robot>

Commit message: intertia added

File: mino_description/urdf/include/common_macros.urdf.xacro (robot description, xacro)
@@ -8,4 +8,9 @@
     params="link_name:='base_link' base_prop mesh:='' scale:=''">
     <link name="${link_name}">
+    <xacro:box_inertia m="${base_prop['mass']}"
+                       x="${base_prop['x_size']}"
+                       y="${base_prop['y_size']}"
+                       z="${base_prop['z_size']}">
+    </xacro:box_inertia>
     <!-- if no 3d model -->
     <xacro:if value="${mesh == ''}">
@@ -47,4 +52,8 @@
 <xacro:property name="pos_z_joint" value="${wheel_props['z_offset']}"/>
     <link name="${prefix}_wheel">
+    <xacro:cylinder_inertia m="${wheel_props['mass']}"
+                            r="${wheel_props['radius']}"
+                            l="${wheel_props['length']}">
+    </xacro:cylinder_inertia>
     <!-- if no 3d model -->
     <xacro:if value="${wheel_props['mesh'] == ''}">
@@ -76,4 +85,7 @@
     params="link_name:='caster_link' caster_props">
     <link name="${link_name}">
+    <xacro:sphere_inertia m="${caster_props['mass']}"
+                          r="${caster_props['radius']}">
+    </xacro:sphere_inertia>
     <xacro:if value="${caster_props['mesh'] == ''}">
         <visual>
@@ -100,3 +112,36 @@
 </xacro:macro>
 <!--##########################################-->
+<!--               Box inertia                -->
+<xacro:macro name="box_inertia" params="m x y z">
+    <inertial>
+        <mass value="${m}"/>
+        <inertia ixx="${m / 12.0 * (y*y + z*z)}" ixy="0.0" ixz="0.0"
+                 iyy="${m / 12.0 * (x*x + z*z)}" iyz="0.0"
+                 izz="${m / 12.0 * (x*x + y*y)}"/>
+        <origin xyz="0.0 0.0 0.0" rpy="0.0 0.0 0.0"/>
+    </inertial>
+</xacro:macro>
+<!--##########################################-->
+<!--            Cylinder inertia              -->
+<xacro:macro name="cylinder_inertia" params="m r l">
+    <inertial>
+        <mass value="${m}"/>
+        <inertia ixx="${m * (3*r*r + l*l) / 12.0}" ixy="0.0" ixz="0.0"
+                 iyy="${m * (3*r*r + l*l) / 12.0}" iyz="0.0"
+                 izz="${m * r*r / 2.0}"/>
+        <origin xyz="0.0 0.0 0.0" rpy="${pi/2} 0.0 0.0"/>
+    </inertial>
+</xacro:macro>
+<!--##########################################-->
+<!--             Sphere inertia               -->
+<xacro:macro name="sphere_inertia" params="m r">
+    <inertial>
+        <mass value="${m}"/>
+        <inertia ixx="${2.0 * m * (r*r) / 5.0}" ixy="0.0" ixz="0.0"
+                 iyy="${2.0 * m * (r*r) / 5.0}" iyz="0.0"
+                 izz="${2.0 * m * (r*r) / 5.0}"/>
+        <origin xyz="0.0 0.0 0.0" rpy="0.0 0.0 0.0"/>
+    </inertial>
+</xacro:macro>
+<!--##########################################-->
 </robot>

Commit message: lidar added

File: mino_description/urdf/include/common_macros.urdf.xacro (robot description, xacro)
@@ -112,4 +112,36 @@
 </xacro:macro>
 <!--##########################################-->
+<!--               Lidar xacro                -->
+<xacro:macro name="lidar"
+    params="link_name:='lidar_link' lidar_props">
+    <link name="${link_name}">
+    <xacro:cylinder_inertia m="${lidar_props['mass']}"
+                            r="${lidar_props['radius']}"
+                            l="${lidar_props['length']}">
+    </xacro:cylinder_inertia>
+    <xacro:if value="${lidar_props['mesh'] == ''}">
+        <visual>
+            <origin xyz="0.0 0.0 0.0" rpy="0.0 0.0 0.0"/>
+            <geometry>
+                <cylinder radius="${lidar_props['radius']}" length="${lidar_props['length']}"/>
+            </geometry>
+            <material name="red"/>
+        </visual>
+        <collision>
+            <origin xyz="0.0 0.0 0.0" rpy="0.0 0.0 0.0"/>
+            <geometry>
+                <cylinder radius="${lidar_props['radius']}" length="${lidar_props['length']}"/>
+            </geometry>
+        </collision>
+    </xacro:if>
+    </link>
+    <joint name="lidar_joint" type="fixed">
+        <parent link="base_link"/>
+        <child link="${link_name}"/>
+        <origin xyz="${lidar_props['x_offset']} ${lidar_props['y_offset']} ${lidar_props['z_offset']}"
+                rpy="0.0 0.0 0.0"/>
+    </joint>
+</xacro:macro>
+<!--##########################################-->
 <!--               Box inertia                -->
 <xacro:macro name="box_inertia" params="m x y z">

File: mino_description/urdf/mino.urdf.xacro (robot description, xacro)
@@ -16,4 +16,6 @@
     <xacro:property name="caster_yaml" value="$(arg config_dir)/caster.yaml"/>
     <xacro:property name="caster_props" value="${xacro.load_yaml(caster_yaml)}"/>
+    <xacro:property name="lidar_yaml" value="$(arg config_dir)/lidar.yaml"/>
+    <xacro:property name="lidar_props" value="${xacro.load_yaml(lidar_yaml)}"/>
     <!-- ########################################## -->
     <!-- Footprint link-->
@@ -27,3 +29,4 @@
     <xacro:caster link_name="caster_link" caster_props="${caster_props}"/>
     <!-- Sensor link -->
+    <xacro:lidar link_name="lidar_link" lidar_props="${lidar_props}"/>
 </robot>

File: mino_gz/urdf/mino_gz.urdf.xacro (robot description, xacro)
@@ -5,4 +5,26 @@
         <mu1 value="0.001"/>
         <mu2 value="0.001"/>
+    </gazebo>
+    <gazebo reference="lidar_link">
+        <sensor name="lidar_sensor" type="gpu_lidar">
+            <gz_frame_id>lidar_link</gz_frame_id>
+            <lidar>
+                <scan>
+                    <horizontal>
+                        <samples>100</samples>
+                        <min_angle>-3.14</min_angle>
+                        <max_angle>3.14</max_angle>
+                    </horizontal>
+                </scan>
+                <range>
+                    <min>0.20</min>
+                    <max>12.0</max>
+                </range>
+            </lidar>
+            <topic>scan</topic>
+            <plugin filename="gz-sim-sensors-system" name="gz::sim::systems::Sensors">
+                <render_engine>ogre2</render_engine>
+            </plugin>
+        </sensor>
     </gazebo>
     <ros2_control name="GazeboSimSystem" type="system">
